File: progettoeagle/progettoeagle.kicad_sch (KiCad schematic)
At the start: 6 parts, among them U1 ACS781LLRTR-100U-T, U2 AD633JRZ-R7, U3 MCP6002-E_P, U4 LM393D, U5 MAX256ASAT

Commit message: Descrizione breve del cambiamento
Parts:
- added D1, D2, D3: AA3527ASESK_J3-50MAV, AA3527ASESK_J3-50MAV:LED_AA3527ASESK_J3-50MAV, symbol AA3527ASESK_J3-50MAV:AA3527ASESK_J3-50MAV
- added J1: Jack-DC, symbol Connector:Jack-DC
- added PS2: R-78AA5.0-1.0SMD-R, R-78AA5.0-1.0SMD-R:CONV_R-78AA5.0-1.0SMD-R, symbol R-78AA5.0-1.0SMD-R:R-78AA5.0-1.0SMD-R
- added R1, R2: ERJU01J221C, ERJU01J221C:RES_ERJU01J221C, symbol ERJU01J221C:ERJU01J221C
- added U6: LTC3202EMS_PBF, LTC3202EMS_PBF:MSOP-10_MS, symbol LTC3202EMS_PBF:LTC3202EMS_PBF
- added U7: MCP6001T-E_LT, MCP6001T-E_LT:SOT65P210X110-5N, symbol MCP6001T-E_LT:MCP6001T-E_LT
Connections:
- new net: D1.1, D1.3, D1.4
- new net: PS2.1 (+VIN), PS2.2 (+VIN)
- new net: PS2.3 (GND), PS2.7 (GND), PS2.8 (GND), PS2.9 (GND)
- new net: PS2.4 (+VOUT), PS2.5 (+VOUT)
- new net: D3.1, D3.3, D3.4
- new net: D2.1, D2.3, D2.4
